File: KBD8X-MK2.kicad_pcb (KiCad board)
At the start: 2 copper layers, 343.7 x 118.3 mm, 347 parts, among them J1 AVR-ISP-6, Q1 DSS60601MZ4-13, SW1 SW_Push, SW2 SW_SPDT, SW3 SW_SPDT, U1 ATmega32U4-MU, U2 PRTR5V0U2X, Y1 16MHz

Commit message: Convert project to KiCad 6 format
Other:
- outline, holes or cut-outs redrawn
- net class Default removed
- net class Power removed
